File: moofpico.kicad_sch (KiCad schematic)
At the start: 19 parts, among them J100 Bus_Apple_II_Card_Side, J2 Micro_SD_Card_Det2, Q1 BS170, U2 74F11, U3 74LVC245, U4 74LVC245, U5 74LVC245, U6 RaspberryPi_Pico

Commit message: add (unpopulated) reset button for pico; fix direction of IRQ (NFCI)
Parts:
- added SW1: SW_SPST, Connector_PinSocket_1.27mm:PinSocket_1x02_P1.27mm_Vertical, symbol Switch:SW_SPST
Connections:
- net GND: now also SW1.1 (A)
- net at U6.30 (RUN): now also SW1.2 (B)
- no-connect marks 28 -> 27
Changed lines of the file:
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@@
 	(title_block
 		(title "moofpico")
-		(rev "0.1")
+		(rev "0.2")
 	)
 	(junction
@@
 	)
 	(no_connect
-		(at 99.06 80.01)
-	)
-	(no_connect
 		(at 134.62 190.5)
 	)
@@
 	(wire
 		(pts
+			(xy 87.63 78.74) (xy 97.79 78.74)
+		)
+		(stroke
+			(width 0)
+			(type default)
+		)
+	)
+	(wire
+		(pts
 			(xy 219.71 140.97) (xy 219.71 143.51)
 		)
@@
 	(wire
 		(pts
+			(xy 97.79 78.74) (xy 99.06 80.01)
+		)
+		(stroke
+			(width 0)
+			(type default)
+		)
+	)
+	(wire
+		(pts
 			(xy 161.29 49.53) (xy 179.07 49.53)
 		)
@@
 	(text "Internally pulled high"
 		(exclude_from_sim no)
-		(at 88.392 81.28 0)
+		(at 91.948 84.328 0)
 		(effects
 			(font
@@
 	)
 	(global_label "TTL{slash}RES"
-		(shape input)
+		(shape output)
 		(at 148.59 170.18 0)
 		(fields_autoplaced yes)
@@
 	)
 	(symbol
+		(lib_id "Switch:SW_SPST")
+		(at 82.55 78.74 0)
+		(unit 1)
+		(exclude_from_sim no)
+		(in_bom yes)
+		(on_board yes)
+		(dnp yes)
+		(property "Reference" "SW1"
+			(at 82.55 72.39 0)
+			(effects
+				(font
+					(size 1.27 1.27)
+				)
+				(hide yes)
+			)
+		)
+		(property "Value" "SW_SPST"
+			(at 82.55 74.93 0)
+			(effects
+				(font
+					(size 1.27 1.27)
+				)
+				(hide yes)
+			)
+		)
+		(property "Footprint" "Connector_PinSocket_1.27mm:PinSocket_1x02_P1.27mm_Vertical"
+			(at 82.55 78.74 0)
+			(effects
+				(font
+					(size 1.27 1.27)
+				)
+				(hide yes)
+			)
+		)
+		(property "Datasheet" "~"
+			(at 82.55 78.74 0)
+			(effects
+				(font
+					(size 1.27 1.27)
+				)
+				(hide yes)
+			)
+		)
+		(property "Description" "Reset Pico"
+			(at 82.55 80.264 0)
+			(effects
+				(font
+					(size 1.27 1.27)
+				)
+			)
+		)
+		(pin "2"
+		)
+		(pin "1"
+		)
+		(instances
+			(project "moofpico"
+				(path "/adf04048-7c47-4d7c-943c-c55ccf696419"
+					(reference "SW1")
+					(unit 1)
+				)
+			)
+		)
+	)
+	(symbol
 		(lib_id "power:GND")
 		(at 198.12 163.83 0)
@@
 					(unit 1)
 				)
+			)
+		)
+	)
+	(symbol
+		(lib_id "power:GND")
+		(at 77.47 78.74 270)
+		(unit 1)
+		(exclude_from_sim no)
+		(in_bom yes)
+		(on_board yes)
+		(dnp no)
+		(fields_autoplaced yes)
+		(property "Reference" "#PWR02"
+			(at 71.12 78.74 0)
+			(effects
+				(font
+					(size 1.27 1.27)
+				)
+				(hide yes)
+			)
+		)
+		(property "Value" "GND"
+			(at 73.66 78.7399 90)
+			(effects
+				(font
+					(size 1.27 1.27)
+				)
+				(justify right)
+			)
+		)
+		(property "Footprint" ""
+			(at 77.47 78.74 0)
+			(effects
+				(font
+					(size 1.27 1.27)
+				)
+				(hide yes)
+			)
+		)
+		(property "Datasheet" ""
+			(at 77.47 78.74 0)
+			(effects
+				(font
+					(size 1.27 1.27)
+				)
+				(hide yes)
+			)
+		)
+		(property "Description" "Power symbol creates a global label with name \"GND\" , ground"
+			(at 77.47 78.74 0)
+			(effects
+				(font
+					(size 1.27 1.27)
+				)
+				(hide yes)
+			)
+		)
+		(pin "1"
+		)
+		(instances
+			(project "moofpico"
+				(path "/adf04048-7c47-4d7c-943c-c55ccf696419"
+					(reference "#PWR02")
+					(unit 1)
+				)

Commit message: updated pi and apple II slots; NFCI
Connections:
- no-connect marks 27 -> 28
Changed lines of the file:
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@@
+	)
+	(no_connect
+		(at 144.78 149.86)
 	)
 	(no_connect
